Commit message: update hardware

File: crane_x7_description/urdf/crane_x7.urdf.xacro (robot description, xacro)
@@ -47,5 +47,5 @@
   <xacro:property name="NAME_JOINT_6" value="crane_x7_lower_arm_revolute_part_joint"/>
   <xacro:property name="NAME_JOINT_7" value="crane_x7_wrist_joint"/>
-  <xacro:property name="NAME_JOINT_HAND" value="crane_x7_gripper_finger_a_joint_trans"/>
+  <xacro:property name="NAME_JOINT_HAND" value="crane_x7_gripper_finger_a_joint"/>
   <xacro:property name="NAME_LINK_BASE" value="crane_x7_shoulder_fixed_part_link"/>
   <xacro:property name="NAME_LINK_1" value="crane_x7_shoulder_revolute_part_link"/>
