Commit message: update

File: crane_x7_description/urdf/crane_x7.gazebo.xacro (robot description, xacro)
@@ -10,5 +10,4 @@
             name_link_6
             name_link_hand">
-<!--
     <gazebo>
       <plugin filename="libgazebo_ros2_control.so" name="gazebo_ros2_control">
@@ -16,6 +15,5 @@
         <parameters>$(find crane_x7_control)/config/crane_x7_controllers.yaml</parameters>
       </plugin>
-    </gazebo> -->
-<!--
+    </gazebo>
     <gazebo reference="${name_link_base}">
       <material>Gazebo/Red</material>
@@ -41,5 +39,5 @@
     <gazebo reference="${name_link_hand}">
       <material>Gazebo/Red</material>
-    </gazebo> -->
+    </gazebo>
   </xacro:macro>
 </robot>

File: crane_x7_description/urdf/crane_x7.gazebo_ros2_control.xacro (robot description, xacro)
@@ -18,6 +18,6 @@
       <joint name="${name_joint_1}">
         <command_interface name="${control_mode}">
-          <param name="min">"-10.0"</param>
-          <param name="max">"10.0"</param>
+          <param name="min">-10.0</param>
+          <param name="max">10.0</param>
         </command_interface>
         <state_interface name="position"/>
@@ -27,6 +27,6 @@
       <joint name="${name_joint_2}">
         <command_interface name="${control_mode}">
-          <param name="min">"-10.0"</param>
-          <param name="max">"10.0"</param>
+          <param name="min">-10.0</param>
+          <param name="max">10.0</param>
         </command_interface>
         <state_interface name="position"/>
@@ -36,6 +36,6 @@
       <joint name="${name_joint_3}">
         <command_interface name="${control_mode}">
-          <param name="min">"-4.0"</param>
-          <param name="max">"4.0"</param>
+          <param name="min">-4.0</param>
+          <param name="max">4.0</param>
         </command_interface>
         <state_interface name="position"/>
@@ -45,6 +45,6 @@
       <joint name="${name_joint_4}">
         <command_interface name="${control_mode}">
-          <param name="min">"-4.0"</param>
-          <param name="max">"4.0"</param>
+          <param name="min">-4.0</param>
+          <param name="max">4.0</param>
         </command_interface>
         <state_interface name="position"/>
@@ -54,6 +54,6 @@
       <joint name="${name_joint_5}">
         <command_interface name="${control_mode}">
-          <param name="min">"-4.0"</param>
-          <param name="max">"4.0"</param>
+          <param name="min">-4.0</param>
+          <param name="max">4.0</param>
         </command_interface>
         <state_interface name="position"/>
@@ -63,6 +63,6 @@
       <joint name="${name_joint_6}">
         <command_interface name="${control_mode}">
-          <param name="min">"-4.0"</param>
-          <param name="max">"4.0"</param>
+          <param name="min">-4.0</param>
+          <param name="max">4.0</param>
         </command_interface>
         <state_interface name="position"/>
@@ -72,6 +72,6 @@
       <joint name="${name_joint_7}">
         <command_interface name="${control_mode}">
-          <param name="min">"-4.0"</param>
-          <param name="max">"4.0"</param>
+          <param name="min">-4.0</param>
+          <param name="max">4.0</param>
         </command_interface>
         <state_interface name="position"/>
@@ -81,6 +81,6 @@
       <joint name="${name_joint_hand}">
         <command_interface name="${control_mode}">
-          <param name="min">"-4.0"</param>
-          <param name="max">"4.0"</param>
+          <param name="min">-4.0</param>
+          <param name="max">4.0</param>
         </command_interface>
         <state_interface name="position"/>

File: crane_x7_description/urdf/crane_x7.ros2_control.xacro (robot description, xacro)
@@ -110,5 +110,5 @@
       </joint>
       <joint name="${name_joint_hand}">
-        <command_interface name="${control_mode}">
+        <command_interface name="effort">
           <param name="min">${vmax}</param>
           <param name="max">${vmin}</param>

File: crane_x7_description/urdf/crane_x7.urdf.xacro (robot description, xacro)
@@ -47,5 +47,5 @@
   <xacro:property name="NAME_JOINT_6" value="crane_x7_lower_arm_revolute_part_joint"/>
   <xacro:property name="NAME_JOINT_7" value="crane_x7_wrist_joint"/>
-  <xacro:property name="NAME_JOINT_HAND" value="crane_x7_joint_hand"/>
+  <xacro:property name="NAME_JOINT_HAND" value="crane_x7_gripper_finger_a_joint_trans"/>
   <xacro:property name="NAME_LINK_BASE" value="crane_x7_shoulder_fixed_part_link"/>
   <xacro:property name="NAME_LINK_1" value="crane_x7_shoulder_revolute_part_link"/>
@@ -58,5 +58,5 @@
   <xacro:unless value="$(arg use_gazebo)">
     <xacro:crane_x7_ros2_control_settings
-      name="crane_plus"
+      name="crane_x7"
       name_joint_1="${NAME_JOINT_1}"
       name_joint_2="${NAME_JOINT_2}"
@@ -79,5 +79,5 @@
       name_link_hand="${NAME_LINK_HAND}"/>
     <xacro:crane_x7_gazebo_ros2_control_settings
-      name="crane_plus"
+      name="crane_x7"
       name_joint_1="${NAME_JOINT_1}"
       name_joint_2="${NAME_JOINT_2}"

Commit message: reconfigure pkg

File: crane_x7_description/urdf/crane_x7.gazebo.xacro (robot description, xacro)
@@ -12,5 +12,5 @@
     <gazebo>
       <plugin filename="libgazebo_ros2_control.so" name="gazebo_ros2_control">
-        <robot_sim_type>gazebo_ros2_control/GazeboSystem</robot_sim_type>
+        <!-- <robot_sim_type>gazebo_ros2_control/GazeboSystem</robot_sim_type> -->
         <parameters>$(find crane_x7_gazebo)/config/crane_x7_gazebo_controllers.yaml</parameters>
       </plugin>

File: crane_x7_description/urdf/crane_x7.gazebo_ros2_control.xacro (robot description, xacro)
@@ -11,9 +11,9 @@
             name_joint_7
             name_joint_hand">
-    <xacro:property name="control_mode" value="effort"/>
     <ros2_control name="${name}" type="system">
       <hardware>
         <plugin>gazebo_ros2_control/GazeboSystem</plugin>
       </hardware>
+      <xacro:property name="control_mode" value="effort"/>
       <joint name="${name_joint_1}">
         <command_interface name="${control_mode}">

File: crane_x7_description/urdf/crane_x7.ros2_control.xacro (robot description, xacro)
@@ -11,20 +11,17 @@
             name_joint_7
             name_joint_hand">
-    <xacro:property name="control_mode" value="velocity"/>
-    <xacro:property name="vmax" value="4.81710873"/>
-    <xacro:property name="vmin" value="-4.81710873"/>
     <ros2_control name="${name}" type="system">
       <hardware>
-        <plugin>crane_x7_hardware/CraneX7Hardware</plugin>
-        <param name="port_name">/dev/ttyUSB0</param>
-        <param name="baudrate">3000000</param>
-        <param name="timeout_seconds">5.0</param>
-        <param name="read_velocities">0</param>
-        <param name="read_loads">0</param>
-        <param name="read_voltages">0</param>
-        <param name="read_temperatures">0</param>
+        <plugin>dynamixel_hardware/DynamixelHardware</plugin>
+        <param name="usb_port">/dev/ttyUSB0</param>
+        <param name="baud_rate">3000000</param>
+        <param name="joint_ids">2, 3, 4, 5, 6, 7, 8, 9</param>
+        <!-- <param name="use_dummy">true</param> -->
       </hardware>
+      <xacro:property name="vmax" value="4.81710873"/>
+      <xacro:property name="vmin" value="-4.81710873"/>
       <joint name="${name_joint_1}">
-        <command_interface name="${control_mode}">
+        <command_interface name="position"/>
+        <command_interface name="velocity">
           <param name="min">${vmax}</param>
           <param name="max">${vmin}</param>
@@ -32,11 +29,10 @@
         <state_interface name="position"/>
         <state_interface name="velocity"/>
-        <state_interface name="load"/>
-        <state_interface name="voltage"/>
-        <state_interface name="temperature"/>
+        <state_interface name="effort"/>
         <param name="dxl_id">2</param>
       </joint>
       <joint name="${name_joint_2}">
-        <command_interface name="${control_mode}">
+        <command_interface name="position"/>
+        <command_interface name="velocity">
           <param name="min">${vmax}</param>
           <param name="max">${vmin}</param>
@@ -44,11 +40,10 @@
         <state_interface name="position"/>
         <state_interface name="velocity"/>
-        <state_interface name="load"/>
-        <state_interface name="voltage"/>
-        <state_interface name="temperature"/>
+        <state_interface name="effort"/>
         <param name="dxl_id">3</param>
       </joint>
       <joint name="${name_joint_3}">
-        <command_interface name="${control_mode}">
+        <command_interface name="position"/>
+        <command_interface name="velocity">
           <param name="min">${vmax}</param>
           <param name="max">${vmin}</param>
@@ -56,11 +51,10 @@
         <state_interface name="position"/>
         <state_interface name="velocity"/>
-        <state_interface name="load"/>
-        <state_interface name="voltage"/>
-        <state_interface name="temperature"/>
+        <state_interface name="effort"/>
         <param name="dxl_id">4</param>
       </joint>
       <joint name="${name_joint_4}">
-        <command_interface name="${control_mode}">
+        <command_interface name="position"/>
+        <command_interface name="velocity">
           <param name="min">${vmax}</param>
           <param name="max">${vmin}</param>
@@ -68,11 +62,10 @@
         <state_interface name="position"/>
         <state_interface name="velocity"/>
-        <state_interface name="load"/>
-        <state_interface name="voltage"/>
-        <state_interface name="temperature"/>
+        <state_interface name="effort"/>
         <param name="dxl_id">5</param>
       </joint>
       <joint name="${name_joint_5}">
-        <command_interface name="${control_mode}">
+        <command_interface name="position"/>
+        <command_interface name="velocity">
           <param name="min">${vmax}</param>
           <param name="max">${vmin}</param>
@@ -80,11 +73,10 @@
         <state_interface name="position"/>
         <state_interface name="velocity"/>
-        <state_interface name="load"/>
-        <state_interface name="voltage"/>
-        <state_interface name="temperature"/>
+        <state_interface name="effort"/>
         <param name="dxl_id">6</param>
       </joint>
       <joint name="${name_joint_6}">
-        <command_interface name="${control_mode}">
+        <command_interface name="position"/>
+        <command_interface name="velocity">
           <param name="min">${vmax}</param>
           <param name="max">${vmin}</param>
@@ -92,11 +84,10 @@
         <state_interface name="position"/>
         <state_interface name="velocity"/>
-        <state_interface name="load"/>
-        <state_interface name="voltage"/>
-        <state_interface name="temperature"/>
+        <state_interface name="effort"/>
         <param name="dxl_id">7</param>
       </joint>
       <joint name="${name_joint_7}">
-        <command_interface name="${control_mode}">
+        <command_interface name="position"/>
+        <command_interface name="velocity">
           <param name="min">${vmax}</param>
           <param name="max">${vmin}</param>
@@ -104,11 +95,10 @@
         <state_interface name="position"/>
         <state_interface name="velocity"/>
-        <state_interface name="load"/>
-        <state_interface name="voltage"/>
-        <state_interface name="temperature"/>
+        <state_interface name="effort"/>
         <param name="dxl_id">8</param>
       </joint>
       <joint name="${name_joint_hand}">
-        <command_interface name="effort">
+        <command_interface name="position"/>
+        <command_interface name="velocity">
           <param name="min">${vmax}</param>
           <param name="max">${vmin}</param>
@@ -116,7 +106,5 @@
         <state_interface name="position"/>
         <state_interface name="velocity"/>
-        <state_interface name="load"/>
-        <state_interface name="voltage"/>
-        <state_interface name="temperature"/>
+        <state_interface name="effort"/>
         <param name="dxl_id">9</param>
       </joint>

File: crane_x7_description/urdf/crane_x7.urdf.xacro (robot description, xacro)
@@ -39,5 +39,9 @@
     <origin xyz="0 0 0"/>
   </xacro:crane_x7>
-  <xacro:property name="NAME_JOINT_BASE" value="crane_x7_shoulder_fixed_part_mount_joint"/>
+  <!-- Include Gazebo and ros2_control macros -->
+  <xacro:include filename="$(find crane_x7_description)/urdf/crane_x7.ros2_control.xacro"/>
+  <xacro:include filename="$(find crane_x7_description)/urdf/crane_x7.gazebo.xacro"/>
+  <xacro:include filename="$(find crane_x7_description)/urdf/crane_x7.gazebo_ros2_control.xacro"/>
+  <!-- <xacro:property name="NAME_JOINT_BASE" value="crane_x7_shoulder_fixed_part_mount_joint"/>
   <xacro:property name="NAME_JOINT_1" value="crane_x7_shoulder_fixed_part_pan_joint"/>
   <xacro:property name="NAME_JOINT_2" value="crane_x7_shoulder_revolute_part_tilt_joint"/>
@@ -46,7 +50,7 @@
   <xacro:property name="NAME_JOINT_5" value="crane_x7_lower_arm_fixed_part_joint"/>
   <xacro:property name="NAME_JOINT_6" value="crane_x7_lower_arm_revolute_part_joint"/>
-  <xacro:property name="NAME_JOINT_7" value="crane_x7_wrist_joint"/>
+  <xacro:property name="NAME_JOINT_7" value="crane_x7_wrist_joint"/> -->
   <xacro:property name="NAME_JOINT_HAND" value="crane_x7_gripper_finger_a_joint"/>
-  <xacro:property name="NAME_LINK_BASE" value="crane_x7_shoulder_fixed_part_link"/>
+  <!-- <xacro:property name="NAME_LINK_BASE" value="crane_x7_shoulder_fixed_part_link"/>
   <xacro:property name="NAME_LINK_1" value="crane_x7_shoulder_revolute_part_link"/>
   <xacro:property name="NAME_LINK_2" value="crane_x7_upper_arm_fixed_part_link"/>
@@ -54,5 +58,5 @@
   <xacro:property name="NAME_LINK_4" value="crane_x7_lower_arm_fixed_part_link"/>
   <xacro:property name="NAME_LINK_5" value="crane_x7_lower_arm_revolute_part_link"/>
-  <xacro:property name="NAME_LINK_6" value="crane_x7_wrist_link"/>
+  <xacro:property name="NAME_LINK_6" value="crane_x7_wrist_link"/> -->
   <xacro:property name="NAME_LINK_HAND" value="crane_x7_wide_two_finger_gripper"/>
   <xacro:unless value="$(arg use_gazebo)">

File: crane_x7_description/urdf/crane_x7.xacro (robot description, xacro)
@@ -4,7 +4,4 @@
   <xacro:include filename="$(find crane_x7_description)/urdf/crane_x7_arm.xacro"/>
   <xacro:include filename="$(find crane_x7_description)/urdf/crane_x7_wide_two_finger_gripper.xacro"/>
-  <xacro:include filename="$(find crane_x7_description)/urdf/crane_x7.ros2_control.xacro"/>
-  <xacro:include filename="$(find crane_x7_description)/urdf/crane_x7.gazebo.xacro"/>
-  <xacro:include filename="$(find crane_x7_description)/urdf/crane_x7.gazebo_ros2_control.xacro"/>
   <material name="black">
     <color rgba="0.2 0.2 0.2 1.0"/>

Commit message: update

File: crane_x7_description/urdf/crane_x7.gazebo.xacro (robot description, xacro)
@@ -12,5 +12,5 @@
     <gazebo>
       <plugin filename="libgazebo_ros2_control.so" name="gazebo_ros2_control">
-        <!-- <robot_sim_type>gazebo_ros2_control/GazeboSystem</robot_sim_type> -->
+        <robot_sim_type>gazebo_ros2_control/GazeboSystem</robot_sim_type>
         <parameters>$(find crane_x7_gazebo)/config/crane_x7_gazebo_controllers.yaml</parameters>
       </plugin>

File: crane_x7_description/urdf/crane_x7.gazebo_ros2_control.xacro (robot description, xacro)
@@ -13,78 +13,73 @@
     <ros2_control name="${name}" type="system">
       <hardware>
-        <plugin>gazebo_ros2_control/GazeboSystem</plugin>
+        <!-- <plugin>gazebo_ros2_control/GazeboSystem</plugin> -->
+        <plugin>test_system</plugin>
       </hardware>
-      <xacro:property name="control_mode" value="effort"/>
+      <xacro:property name="control_mode" value="velocity"/>
+      <xacro:property name="vmax" value="4.81710873"/>
+      <xacro:property name="vmin" value="-4.81710873"/>
       <joint name="${name_joint_1}">
         <command_interface name="${control_mode}">
-          <param name="min">-10.0</param>
-          <param name="max">10.0</param>
+          <param name="min">${vmax}</param>
+          <param name="max">${vmin}</param>
         </command_interface>
         <state_interface name="position"/>
         <state_interface name="velocity"/>
-        <state_interface name="effort"/>
       </joint>
       <joint name="${name_joint_2}">
         <command_interface name="${control_mode}">
-          <param name="min">-10.0</param>
-          <param name="max">10.0</param>
+          <param name="min">${vmax}</param>
+          <param name="max">${vmin}</param>
         </command_interface>
         <state_interface name="position"/>
         <state_interface name="velocity"/>
-        <state_interface name="effort"/>
       </joint>
       <joint name="${name_joint_3}">
         <command_interface name="${control_mode}">
-          <param name="min">-4.0</param>
-          <param name="max">4.0</param>
+          <param name="min">${vmax}</param>
+          <param name="max">${vmin}</param>
         </command_interface>
         <state_interface name="position"/>
         <state_interface name="velocity"/>
-        <state_interface name="effort"/>
       </joint>
       <joint name="${name_joint_4}">
         <command_interface name="${control_mode}">
-          <param name="min">-4.0</param>
-          <param name="max">4.0</param>
+          <param name="min">${vmax}</param>
+          <param name="max">${vmin}</param>
         </command_interface>
         <state_interface name="position"/>
         <state_interface name="velocity"/>
-        <state_interface name="effort"/>
       </joint>
       <joint name="${name_joint_5}">
         <command_interface name="${control_mode}">
-          <param name="min">-4.0</param>
-          <param name="max">4.0</param>
+          <param name="min">${vmax}</param>
+          <param name="max">${vmin}</param>
         </command_interface>
         <state_interface name="position"/>
         <state_interface name="velocity"/>
-        <state_interface name="effort"/>
       </joint>
       <joint name="${name_joint_6}">
         <command_interface name="${control_mode}">
-          <param name="min">-4.0</param>
-          <param name="max">4.0</param>
+          <param name="min">${vmax}</param>
+          <param name="max">${vmin}</param>
         </command_interface>
         <state_interface name="position"/>
         <state_interface name="velocity"/>
-        <state_interface name="effort"/>
       </joint>
       <joint name="${name_joint_7}">
         <command_interface name="${control_mode}">
-          <param name="min">-4.0</param>
-          <param name="max">4.0</param>
+          <param name="min">${vmax}</param>
+          <param name="max">${vmin}</param>
         </command_interface>
         <state_interface name="position"/>
         <state_interface name="velocity"/>
-        <state_interface name="effort"/>
       </joint>
       <joint name="${name_joint_hand}">
         <command_interface name="${control_mode}">
-          <param name="min">-4.0</param>
-          <param name="max">4.0</param>
+          <param name="min">${vmax}</param>
+          <param name="max">${vmin}</param>
         </command_interface>
         <state_interface name="position"/>
         <state_interface name="velocity"/>
-        <state_interface name="effort"/>
       </joint>
     </ros2_control>

File: crane_x7_description/urdf/crane_x7.ros2_control.xacro (robot description, xacro)
@@ -17,5 +17,4 @@
         <param name="baud_rate">3000000</param>
         <param name="joint_ids">2, 3, 4, 5, 6, 7, 8, 9</param>
-        <!-- <param name="use_dummy">true</param> -->
       </hardware>
       <xacro:property name="vmax" value="4.81710873"/>
@@ -29,6 +28,4 @@
         <state_interface name="position"/>
         <state_interface name="velocity"/>
-        <state_interface name="effort"/>
-        <param name="dxl_id">2</param>
       </joint>
       <joint name="${name_joint_2}">
@@ -40,6 +37,4 @@
         <state_interface name="position"/>
         <state_interface name="velocity"/>
-        <state_interface name="effort"/>
-        <param name="dxl_id">3</param>
       </joint>
       <joint name="${name_joint_3}">
@@ -51,6 +46,4 @@
         <state_interface name="position"/>
         <state_interface name="velocity"/>
-        <state_interface name="effort"/>
-        <param name="dxl_id">4</param>
       </joint>
       <joint name="${name_joint_4}">
@@ -62,6 +55,4 @@
         <state_interface name="position"/>
         <state_interface name="velocity"/>
-        <state_interface name="effort"/>
-        <param name="dxl_id">5</param>
       </joint>
       <joint name="${name_joint_5}">
@@ -73,6 +64,4 @@
         <state_interface name="position"/>
         <state_interface name="velocity"/>
-        <state_interface name="effort"/>
-        <param name="dxl_id">6</param>
       </joint>
       <joint name="${name_joint_6}">
@@ -84,6 +73,4 @@
         <state_interface name="position"/>
         <state_interface name="velocity"/>
-        <state_interface name="effort"/>
-        <param name="dxl_id">7</param>
       </joint>
       <joint name="${name_joint_7}">
@@ -95,6 +82,4 @@
         <state_interface name="position"/>
         <state_interface name="velocity"/>
-        <state_interface name="effort"/>
-        <param name="dxl_id">8</param>
       </joint>
       <joint name="${name_joint_hand}">
@@ -106,6 +91,4 @@
         <state_interface name="position"/>
         <state_interface name="velocity"/>
-        <state_interface name="effort"/>
-        <param name="dxl_id">9</param>
       </joint>
     </ros2_control>
