Commit message: fix gazebo lanch files

File: crane_x7_description/urdf/crane_x7.gazebo_ros2_control.xacro (robot description, xacro)
@@ -13,6 +13,5 @@
     <ros2_control name="${name}" type="system">
       <hardware>
-        <!-- <plugin>gazebo_ros2_control/GazeboSystem</plugin> -->
-        <plugin>test_system</plugin>
+        <plugin>gazebo_ros2_control/GazeboSystem</plugin>
       </hardware>
       <xacro:property name="control_mode" value="velocity"/>

File: crane_x7_description/urdf/crane_x7_arm.xacro (robot description, xacro)
@@ -57,5 +57,5 @@
         <origin xyz="0 0 0" rpy="0 0 0"/>
         <geometry>
-          <mesh filename="package://crane_x7_description/meshes/visual/base_fixed_part.stl"
+          <mesh filename="file://$(find crane_x7_description)/meshes/visual/base_fixed_part.stl"
               scale="1 1 1"/>
         </geometry>
@@ -65,5 +65,5 @@
         <origin xyz="0 0 0" rpy="0 0 0"/>
         <geometry>
-          <mesh filename="package://crane_x7_description/meshes/collision/base_fixed_part.stl"
+          <mesh filename="file://$(find crane_x7_description)/meshes/collision/base_fixed_part.stl"
               scale="1 1 1"/>
         </geometry>
@@ -105,5 +105,5 @@
         <origin xyz="0 0 0" rpy="0 0 ${M_PI}"/>
         <geometry>
-          <mesh filename="package://crane_x7_description/meshes/visual/base_revolute_part.stl"
+          <mesh filename="file://$(find crane_x7_description)/meshes/visual/base_revolute_part.stl"
               scale="1 1 1"/>
         </geometry>
@@ -113,5 +113,5 @@
         <!--<origin xyz="0 0 0" rpy="0 0 ${M_PI}"/>-->
         <!--<geometry>-->
-          <!--<mesh filename="package://crane_x7_description/meshes/collision/base_revolute_part.stl"-->
+          <!--<mesh filename="file://$(find crane_x7_description)/meshes/collision/base_revolute_part.stl"-->
               <!--scale="1 1 1"/>-->
         <!--</geometry>-->
@@ -163,5 +163,5 @@
         <origin xyz="0 0 0" rpy="${M_PI/2} 0 0"/>
         <geometry>
-          <mesh filename="package://crane_x7_description/meshes/visual/rotating_link_type_1_fixed_part.stl"
+          <mesh filename="file://$(find crane_x7_description)/meshes/visual/rotating_link_type_1_fixed_part.stl"
               scale="1 1 1"/>
         </geometry>
@@ -171,5 +171,5 @@
         <origin xyz="0 0 0" rpy="${M_PI/2} 0 0"/>
         <geometry>
-          <mesh filename="package://crane_x7_description/meshes/collision/rotating_link_type_1_fixed_part.stl"
+          <mesh filename="file://$(find crane_x7_description)/meshes/collision/rotating_link_type_1_fixed_part.stl"
               scale="1 1 1"/>
         </geometry>
@@ -194,5 +194,5 @@
         <origin xyz="0 0 0" rpy="-${M_PI/2} 0 0"/>
         <geometry>
-          <mesh filename="package://crane_x7_description/meshes/visual/joint_cover.stl"
+          <mesh filename="file://$(find crane_x7_description)/meshes/visual/joint_cover.stl"
               scale="1 1 1"/>
         </geometry>
@@ -202,5 +202,5 @@
         <origin xyz="0 0 0" rpy="-${M_PI/2} 0 0"/>
         <geometry>
-          <mesh filename="package://crane_x7_description/meshes/visual/joint_cover.stl"
+          <mesh filename="file://$(find crane_x7_description)/meshes/visual/joint_cover.stl"
               scale="1 1 1"/>
         </geometry>
@@ -218,5 +218,5 @@
         <origin xyz="0 0 0" rpy="${M_PI/2} 0 0"/>
         <geometry>
-          <mesh filename="package://crane_x7_description/meshes/visual/joint_cover.stl"
+          <mesh filename="file://$(find crane_x7_description)/meshes/visual/joint_cover.stl"
               scale="1 1 1"/>
         </geometry>
@@ -226,5 +226,5 @@
         <origin xyz="0 0 0" rpy="${M_PI/2} 0 0"/>
         <geometry>
-          <mesh filename="package://crane_x7_description/meshes/visual/joint_cover.stl"
+          <mesh filename="file://$(find crane_x7_description)/meshes/visual/joint_cover.stl"
               scale="1 1 1"/>
         </geometry>
@@ -262,5 +262,5 @@
         <origin xyz="0 0 0" rpy="0 0 0"/>
         <geometry>
-          <mesh filename="package://crane_x7_description/meshes/visual/rotating_link_type_1_revolute_part.stl"
+          <mesh filename="file://$(find crane_x7_description)/meshes/visual/rotating_link_type_1_revolute_part.stl"
               scale="1 1 1"/>
         </geometry>
@@ -270,5 +270,5 @@
         <origin xyz="0 0 0" rpy="0 0 0"/>
         <geometry>
-          <mesh filename="package://crane_x7_description/meshes/collision/rotating_link_type_1_revolute_part.stl"
+          <mesh filename="file://$(find crane_x7_description)/meshes/collision/rotating_link_type_1_revolute_part.stl"
               scale="1 1 1"/>
         </geometry>
@@ -313,5 +313,5 @@
         <origin xyz="0 0 0" rpy="${M_PI/2} 0 0"/>
         <geometry>
-          <mesh filename="package://crane_x7_description/meshes/visual/rotating_link_type_2_fixed_part.stl"
+          <mesh filename="file://$(find crane_x7_description)/meshes/visual/rotating_link_type_2_fixed_part.stl"
               scale="1 1 1"/>
         </geometry>
@@ -321,5 +321,5 @@
         <origin xyz="0 0 0" rpy="${M_PI/2} 0 0"/>
         <geometry>
-          <mesh filename="package://crane_x7_description/meshes/collision/rotating_link_type_2_fixed_part.stl"
+          <mesh filename="file://$(find crane_x7_description)/meshes/collision/rotating_link_type_2_fixed_part.stl"
               scale="1 1 1"/>
         </geometry>
@@ -344,5 +344,5 @@
         <origin xyz="0 0 0" rpy="-${M_PI/2} 0 0"/>
         <geometry>
-          <mesh filename="package://crane_x7_description/meshes/visual/joint_cover.stl"
+          <mesh filename="file://$(find crane_x7_description)/meshes/visual/joint_cover.stl"
               scale="1 1 1"/>
         </geometry>
@@ -352,5 +352,5 @@
         <origin xyz="0 0 0" rpy="-${M_PI/2} 0 0"/>
         <geometry>
-          <mesh filename="package://crane_x7_description/meshes/visual/joint_cover.stl"
+          <mesh filename="file://$(find crane_x7_description)/meshes/visual/joint_cover.stl"
               scale="1 1 1"/>
         </geometry>
@@ -368,5 +368,5 @@
         <origin xyz="0 0 0" rpy="${M_PI/2} 0 0"/>
         <geometry>
-          <mesh filename="package://crane_x7_description/meshes/visual/joint_cover.stl"
+          <mesh filename="file://$(find crane_x7_description)/meshes/visual/joint_cover.stl"
               scale="1 1 1"/>
         </geometry>
@@ -376,5 +376,5 @@
         <origin xyz="0 0 0" rpy="${M_PI/2} 0 0"/>
         <geometry>
-          <mesh filename="package://crane_x7_description/meshes/visual/joint_cover.stl"
+          <mesh filename="file://$(find crane_x7_description)/meshes/visual/joint_cover.stl"
               scale="1 1 1"/>
         </geometry>
@@ -409,5 +409,5 @@
         <origin xyz="0 0 0" rpy="0 0 0"/>
         <geometry>
-          <mesh filename="package://crane_x7_description/meshes/visual/rotating_link_type_2_revolute_part.stl"
+          <mesh filename="file://$(find crane_x7_description)/meshes/visual/rotating_link_type_2_revolute_part.stl"
               scale="1 1 1"/>
         </geometry>
@@ -417,5 +417,5 @@
         <origin xyz="0 0 0" rpy="0 0 0"/>
         <geometry>
-          <mesh filename="package://crane_x7_description/meshes/collision/rotating_link_type_2_revolute_part.stl"
+          <mesh filename="file://$(find crane_x7_description)/meshes/collision/rotating_link_type_2_revolute_part.stl"
               scale="1 1 1"/>
         </geometry>
@@ -462,5 +462,5 @@
         <origin xyz="0 0 0" rpy="${M_PI/2} 0 0"/>
         <geometry>
-          <mesh filename="package://crane_x7_description/meshes/visual/wrist.stl"
+          <mesh filename="file://$(find crane_x7_description)/meshes/visual/wrist.stl"
               scale="1 1 1"/>
         </geometry>
@@ -470,5 +470,5 @@
         <origin xyz="0 0 0" rpy="${M_PI/2} 0 0"/>
         <geometry>
-          <mesh filename="package://crane_x7_description/meshes/collision/wrist.stl"
+          <mesh filename="file://$(find crane_x7_description)/meshes/collision/wrist.stl"
               scale="1 1 1"/>
         </geometry>

File: crane_x7_description/urdf/crane_x7_mounting_plate.xacro (robot description, xacro)
@@ -15,5 +15,5 @@
         <origin xyz="0 0 0" rpy="0 0 0"/>
         <geometry>
-          <mesh filename="package://crane_x7_description/meshes/visual/mounting_plate.stl"
+          <mesh filename="file://$(find crane_x7_description)/meshes/visual/mounting_plate.stl"
               scale="1 1 1"/>
         </geometry>
@@ -23,5 +23,5 @@
         <origin xyz="0 0 0" rpy="0 0 0"/>
         <geometry>
-          <mesh filename="package://crane_x7_description/meshes/collision/mounting_plate.stl"
+          <mesh filename="file://$(find crane_x7_description)/meshes/collision/mounting_plate.stl"
               scale="1 1 1"/>
         </geometry>

File: crane_x7_description/urdf/crane_x7_rt_logos.xacro (robot description, xacro)
@@ -7,5 +7,5 @@
         <origin xyz="0 0 0" rpy="-${M_PI/2} ${M_PI/2} 0"/>
         <geometry>
-          <mesh filename="package://crane_x7_description/meshes/visual/rtcorp_logo_name.stl"
+          <mesh filename="file://$(find crane_x7_description)/meshes/visual/rtcorp_logo_name.stl"
               scale="1 1 1"/>
         </geometry>
@@ -17,5 +17,5 @@
         <origin xyz="0 0 0" rpy="-${M_PI/2} ${M_PI/2} 0"/>
         <geometry>
-          <mesh filename="package://crane_x7_description/meshes/visual/rtcorp_logo_name.stl"
+          <mesh filename="file://$(find crane_x7_description)/meshes/visual/rtcorp_logo_name.stl"
               scale="1 1 1"/>
         </geometry>
@@ -32,5 +32,5 @@
         <origin xyz="0 0 0" rpy="-${M_PI/2} ${M_PI/2} 0"/>
         <geometry>
-          <mesh filename="package://crane_x7_description/meshes/visual/rtcorp_logo_rabbit.stl"
+          <mesh filename="file://$(find crane_x7_description)/meshes/visual/rtcorp_logo_rabbit.stl"
               scale="1 1 1"/>
         </geometry>
@@ -40,5 +40,5 @@
         <origin xyz="0 0 0" rpy="-${M_PI/2} ${M_PI/2} 0"/>
         <geometry>
-          <mesh filename="package://crane_x7_description/meshes/visual/rtcorp_logo_rabbit.stl"
+          <mesh filename="file://$(find crane_x7_description)/meshes/visual/rtcorp_logo_rabbit.stl"
               scale="1 1 1"/>
         </geometry>
@@ -55,5 +55,5 @@
         <origin xyz="0 0 0" rpy="${M_PI/2} -${M_PI/2} 0"/>
         <geometry>
-          <mesh filename="package://crane_x7_description/meshes/visual/rtcorp_logo_name.stl"
+          <mesh filename="file://$(find crane_x7_description)/meshes/visual/rtcorp_logo_name.stl"
               scale="1 1 1"/>
         </geometry>
@@ -63,5 +63,5 @@
         <origin xyz="0 0 0" rpy="${M_PI/2} -${M_PI/2} 0"/>
         <geometry>
-          <mesh filename="package://crane_x7_description/meshes/visual/rtcorp_logo_name.stl"
+          <mesh filename="file://$(find crane_x7_description)/meshes/visual/rtcorp_logo_name.stl"
               scale="1 1 1"/>
         </geometry>
@@ -78,5 +78,5 @@
         <origin xyz="0 0 0" rpy="${M_PI/2} -${M_PI/2} 0"/>
         <geometry>
-          <mesh filename="package://crane_x7_description/meshes/visual/rtcorp_logo_rabbit.stl"
+          <mesh filename="file://$(find crane_x7_description)/meshes/visual/rtcorp_logo_rabbit.stl"
               scale="1 1 1"/>
         </geometry>
@@ -86,5 +86,5 @@
         <origin xyz="0 0 0" rpy="${M_PI/2} -${M_PI/2} 0"/>
         <geometry>
-          <mesh filename="package://crane_x7_description/meshes/visual/rtcorp_logo_rabbit.stl"
+          <mesh filename="file://$(find crane_x7_description)/meshes/visual/rtcorp_logo_rabbit.stl"
               scale="1 1 1"/>
         </geometry>

File: crane_x7_description/urdf/crane_x7_wide_two_finger_gripper.xacro (robot description, xacro)
@@ -10,5 +10,5 @@
         <origin xyz="0 0 0" rpy="0 0 0"/>
         <geometry>
-          <mesh filename="package://crane_x7_description/meshes/visual/wide_two_finger_gripper_actuator.stl"
+          <mesh filename="file://$(find crane_x7_description)/meshes/visual/wide_two_finger_gripper_actuator.stl"
               scale="1 1 1"/>
         </geometry>
@@ -18,5 +18,5 @@
         <origin xyz="0 0 0" rpy="0 0 0"/>
         <geometry>
-          <mesh filename="package://crane_x7_description/meshes/collision/wide_two_finger_gripper_actuator.stl"
+          <mesh filename="file://$(find crane_x7_description)/meshes/collision/wide_two_finger_gripper_actuator.stl"
               scale="1 1 1"/>
         </geometry>
@@ -66,5 +66,5 @@
         <origin xyz="0 0 0" rpy="${M_PI/2} 0 0"/>
         <geometry>
-          <mesh filename="package://crane_x7_description/meshes/visual/wide_two_finger_gripper_finger_a.stl"
+          <mesh filename="file://$(find crane_x7_description)/meshes/visual/wide_two_finger_gripper_finger_a.stl"
               scale="1 1 1"/>
         </geometry>
@@ -74,5 +74,5 @@
         <origin xyz="0 0 0" rpy="${M_PI/2} 0 0"/>
         <geometry>
-          <mesh filename="package://crane_x7_description/meshes/collision/wide_two_finger_gripper_finger_a.stl"
+          <mesh filename="file://$(find crane_x7_description)/meshes/collision/wide_two_finger_gripper_finger_a.stl"
               scale="1 1 1"/>
         </geometry>
@@ -99,5 +99,5 @@
         <origin xyz="0 0 0" rpy="${M_PI/2} 0 0"/>
         <geometry>
-          <mesh filename="package://crane_x7_description/meshes/visual/wide_two_finger_gripper_finger_b.stl"
+          <mesh filename="file://$(find crane_x7_description)/meshes/visual/wide_two_finger_gripper_finger_b.stl"
               scale="1 1 1"/>
         </geometry>
@@ -107,5 +107,5 @@
         <origin xyz="0 0 0" rpy="${M_PI/2} 0 0"/>
         <geometry>
-          <mesh filename="package://crane_x7_description/meshes/collision/wide_two_finger_gripper_finger_b.stl"
+          <mesh filename="file://$(find crane_x7_description)/meshes/collision/wide_two_finger_gripper_finger_b.stl"
               scale="1 1 1"/>
         </geometry>
