Commit message: modify repo name of robotoc

File: crane_x7_description/urdf/crane_x7.ros2_control.xacro (robot description, xacro)
@@ -22,8 +22,4 @@
       <joint name="${name_joint_1}">
         <command_interface name="position"/>
-        <command_interface name="velocity">
-          <param name="min">${vmax}</param>
-          <param name="max">${vmin}</param>
-        </command_interface>
         <state_interface name="position"/>
         <state_interface name="velocity"/>
@@ -31,8 +27,4 @@
       <joint name="${name_joint_2}">
         <command_interface name="position"/>
-        <command_interface name="velocity">
-          <param name="min">${vmax}</param>
-          <param name="max">${vmin}</param>
-        </command_interface>
         <state_interface name="position"/>
         <state_interface name="velocity"/>
@@ -40,8 +32,4 @@
       <joint name="${name_joint_3}">
         <command_interface name="position"/>
-        <command_interface name="velocity">
-          <param name="min">${vmax}</param>
-          <param name="max">${vmin}</param>
-        </command_interface>
         <state_interface name="position"/>
         <state_interface name="velocity"/>
@@ -49,8 +37,4 @@
       <joint name="${name_joint_4}">
         <command_interface name="position"/>
-        <command_interface name="velocity">
-          <param name="min">${vmax}</param>
-          <param name="max">${vmin}</param>
-        </command_interface>
         <state_interface name="position"/>
         <state_interface name="velocity"/>
@@ -58,8 +42,4 @@
       <joint name="${name_joint_5}">
         <command_interface name="position"/>
-        <command_interface name="velocity">
-          <param name="min">${vmax}</param>
-          <param name="max">${vmin}</param>
-        </command_interface>
         <state_interface name="position"/>
         <state_interface name="velocity"/>
@@ -67,8 +47,4 @@
       <joint name="${name_joint_6}">
         <command_interface name="position"/>
-        <command_interface name="velocity">
-          <param name="min">${vmax}</param>
-          <param name="max">${vmin}</param>
-        </command_interface>
         <state_interface name="position"/>
         <state_interface name="velocity"/>
@@ -76,8 +52,4 @@
       <joint name="${name_joint_7}">
         <command_interface name="position"/>
-        <command_interface name="velocity">
-          <param name="min">${vmax}</param>
-          <param name="max">${vmin}</param>
-        </command_interface>
         <state_interface name="position"/>
         <state_interface name="velocity"/>
@@ -85,8 +57,4 @@
       <joint name="${name_joint_hand}">
         <command_interface name="position"/>
-        <command_interface name="velocity">
-          <param name="min">${vmax}</param>
-          <param name="max">${vmin}</param>
-        </command_interface>
         <state_interface name="position"/>
         <state_interface name="velocity"/>

File: crane_x7_mpc/experiments/crane_x7_description/urdf/crane_x7.gazebo_ros2_control.xacro (robot description, xacro)
@@ -14,43 +14,70 @@
       <hardware>
         <plugin>gazebo_ros2_control/GazeboSystem</plugin>
-        <!-- <plugin>test_system</plugin> -->
+        <!-- <plugin>test_sstem</plugin> -->
       </hardware>
+      <xacro:property name="control_mode" value="velocity"/>
+      <xacro:property name="vmax" value="4.81710873"/>
+      <xacro:property name="vmin" value="-4.81710873"/>
       <joint name="${name_joint_1}">
-        <command_interface name="position"/>
+        <command_interface name="${control_mode}">
+          <param name="min">${vmax}</param>
+          <param name="max">${vmin}</param>
+        </command_interface>
         <state_interface name="position"/>
         <state_interface name="velocity"/>
       </joint>
       <joint name="${name_joint_2}">
-        <command_interface name="position"/>
+        <command_interface name="${control_mode}">
+          <param name="min">${vmax}</param>
+          <param name="max">${vmin}</param>
+        </command_interface>
         <state_interface name="position"/>
         <state_interface name="velocity"/>
       </joint>
       <joint name="${name_joint_3}">
-        <command_interface name="position"/>
+        <command_interface name="${control_mode}">
+          <param name="min">${vmax}</param>
+          <param name="max">${vmin}</param>
+        </command_interface>
         <state_interface name="position"/>
         <state_interface name="velocity"/>
       </joint>
       <joint name="${name_joint_4}">
-        <command_interface name="position"/>
+        <command_interface name="${control_mode}">
+          <param name="min">${vmax}</param>
+          <param name="max">${vmin}</param>
+        </command_interface>
         <state_interface name="position"/>
         <state_interface name="velocity"/>
       </joint>
       <joint name="${name_joint_5}">
-        <command_interface name="position"/>
+        <command_interface name="${control_mode}">
+          <param name="min">${vmax}</param>
+          <param name="max">${vmin}</param>
+        </command_interface>
         <state_interface name="position"/>
         <state_interface name="velocity"/>
       </joint>
       <joint name="${name_joint_6}">
-        <command_interface name="position"/>
+        <command_interface name="${control_mode}">
+          <param name="min">${vmax}</param>
+          <param name="max">${vmin}</param>
+        </command_interface>
         <state_interface name="position"/>
         <state_interface name="velocity"/>
       </joint>
       <joint name="${name_joint_7}">
-        <command_interface name="position"/>
+        <command_interface name="${control_mode}">
+          <param name="min">${vmax}</param>
+          <param name="max">${vmin}</param>
+        </command_interface>
         <state_interface name="position"/>
         <state_interface name="velocity"/>
       </joint>
       <joint name="${name_joint_hand}">
-        <command_interface name="position"/>
+        <command_interface name="${control_mode}">
+          <param name="min">${vmax}</param>
+          <param name="max">${vmin}</param>
+        </command_interface>
         <state_interface name="position"/>
         <state_interface name="velocity"/>

File: crane_x7_mpc/experiments/crane_x7_description/urdf/crane_x7.ros2_control.xacro (robot description, xacro)
@@ -1,5 +1,5 @@
 <?xml version="1.0"?>
 <robot xmlns:xacro="http://www.ros.org/wiki/xacro">
-  <xacro:macro name="crane_x7_gazebo_ros2_control_settings"
+  <xacro:macro name="crane_x7_ros2_control_settings"
     params="name
             name_joint_1
@@ -13,9 +13,17 @@
     <ros2_control name="${name}" type="system">
       <hardware>
-        <plugin>gazebo_ros2_control/GazeboSystem</plugin>
-        <!-- <plugin>test_system</plugin> -->
+        <plugin>dynamixel_hardware/DynamixelHardware</plugin>
+        <param name="usb_port">/dev/ttyUSB0</param>
+        <param name="baud_rate">3000000</param>
+        <param name="joint_ids">2, 3, 4, 5, 6, 7, 8, 9</param>
       </hardware>
+      <xacro:property name="vmax" value="4.81710873"/>
+      <xacro:property name="vmin" value="-4.81710873"/>
       <joint name="${name_joint_1}">
         <command_interface name="position"/>
+        <command_interface name="velocity">
+          <param name="min">${vmax}</param>
+          <param name="max">${vmin}</param>
+        </command_interface>
         <state_interface name="position"/>
         <state_interface name="velocity"/>
@@ -23,4 +31,8 @@
       <joint name="${name_joint_2}">
         <command_interface name="position"/>
+        <command_interface name="velocity">
+          <param name="min">${vmax}</param>
+          <param name="max">${vmin}</param>
+        </command_interface>
         <state_interface name="position"/>
         <state_interface name="velocity"/>
@@ -28,4 +40,8 @@
       <joint name="${name_joint_3}">
         <command_interface name="position"/>
+        <command_interface name="velocity">
+          <param name="min">${vmax}</param>
+          <param name="max">${vmin}</param>
+        </command_interface>
         <state_interface name="position"/>
         <state_interface name="velocity"/>
@@ -33,4 +49,8 @@
       <joint name="${name_joint_4}">
         <command_interface name="position"/>
+        <command_interface name="velocity">
+          <param name="min">${vmax}</param>
+          <param name="max">${vmin}</param>
+        </command_interface>
         <state_interface name="position"/>
         <state_interface name="velocity"/>
@@ -38,4 +58,8 @@
       <joint name="${name_joint_5}">
         <command_interface name="position"/>
+        <command_interface name="velocity">
+          <param name="min">${vmax}</param>
+          <param name="max">${vmin}</param>
+        </command_interface>
         <state_interface name="position"/>
         <state_interface name="velocity"/>
@@ -43,4 +67,8 @@
       <joint name="${name_joint_6}">
         <command_interface name="position"/>
+        <command_interface name="velocity">
+          <param name="min">${vmax}</param>
+          <param name="max">${vmin}</param>
+        </command_interface>
         <state_interface name="position"/>
         <state_interface name="velocity"/>
@@ -48,4 +76,8 @@
       <joint name="${name_joint_7}">
         <command_interface name="position"/>
+        <command_interface name="velocity">
+          <param name="min">${vmax}</param>
+          <param name="max">${vmin}</param>
+        </command_interface>
         <state_interface name="position"/>
         <state_interface name="velocity"/>
@@ -53,4 +85,8 @@
       <joint name="${name_joint_hand}">
         <command_interface name="position"/>
+        <command_interface name="velocity">
+          <param name="min">${vmax}</param>
+          <param name="max">${vmin}</param>
+        </command_interface>
         <state_interface name="position"/>
         <state_interface name="velocity"/>
